File: The-ENDGAME-MX-BAD.kicad_pcb (KiCad board)
At the start: 2 copper layers, 73 parts, among them SW1 SW_Push, SW10 SW_Push, SW11 SW_Push, SW12 SW_Push, SW13 SW_Push, SW14 SW_Push, SW15 SW_Push, SW16 SW_Push, SW17 SW_Push, SW18 SW_Push, SW19 SW_Push, SW2 SW_Push, SW20 SW_Push, SW21 SW_Push, SW22 SW_Push, SW23 SW_Push, SW24 SW_Push, SW25 SW_Push, SW26 SW_Push, SW27 SW_Push, SW28 SW_Push, SW29 SW_Push, SW3 SW_Push, SW30 SW_Push, SW31 SW_Push, SW32 SW_Push, SW33 SW_Push, SW34 SW_Push, SW35 SW_Push, SW36 SW_Push, SW4 SW_Push, SW5 SW_Push, SW6 SW_Push, SW7 SW_Push, SW8 SW_Push, SW9 SW_Push, U1 ProMicro-kbd-34key

Commit message: fast fertig
Parts:
- added J2: Conn_01x02_Female, Connector_JST:JST_SH_BM02B-SRSS-TB_1x02-1MP_P1.00mm_Vertical, B.Cu at (244.1, 54.4)
- added RSW1: SW_Push, Button_Switch_THT:SW_PUSH_6mm, B.Cu at (217.4, 124.1)
- added SW_POWER1: SW_SPDT, Button_Switch_SMD:SW_SPDT_PCM12, B.Cu at (235.2, 55.2)
- D1, D10, D11, D12, D13, D14, D15, D16, D17, D18, D19, D2, D20, D21, D22, D23, D24, D25, D26, D27, D28, D29, D3, D30, D31, D32, D33, D34, D35, D36, D4, D5, D6, D7, D8, D9: moved to B.Cu
- U1: footprint Keebio-Parts:ArduinoProMicro-BackSide -> Keebio-Parts:Elite-C-castellated-24pin-holes
- moved D31 148.9 mm to (57.8, 131.1), turned to 180 degrees
- moved D21 142.0 mm to (53.3, 114.1), turned to 180 degrees
- moved D20 136.2 mm to (244.6, 97.1), turned to 180 degrees
- moved D23 124.5 mm to (89.7, 99.4), turned to 172 degrees
- moved D35 124.0 mm to (195.7, 131.5), turned to -170 degrees
- moved D12 123.3 mm to (72.6, 84.8), turned to 176 degrees
- moved D36 120.8 mm to (240.1, 131.1), turned to 180 degrees
- moved D19 119.7 mm to (225.3, 84.2), turned to -176 degrees
- moved D29 116.4 mm to (226.5, 101.1), turned to -176 degrees
- moved D30 115.5 mm to (244.6, 114.1), turned to 180 degrees
- moved D33 115.2 mm to (124.3, 136.9), turned to 170 degrees
- moved D11 114.3 mm to (53.3, 97.1), turned to 180 degrees
- moved D34 113.1 mm to (173.6, 135.5), turned to -170 degrees
- moved D32 109.4 mm to (102.2, 133.0), turned to 170 degrees
- moved D27 108.3 mm to (190.0, 103.5), turned to -170 degrees
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
Commit message: pcb changes
Parts:
- RSW1: moved to F.Cu
- U1: moved to B.Cu
- moved RSW1 102.0 mm to (144.0, 53.3), turned to 0 degrees
- moved SW_POWER1 101.0 mm to (134.2, 54.6)
- moved J2 85.0 mm to (159.1, 54.5)
- moved U1 16.0 mm to (147.4, 123.4)
- moved SW34 9.40 mm to (173.2, 138.5), turned to 12 degrees
- moved D34 9.21 mm to (178.7, 143.1), turned to -168 degrees
- moved D7 8.70 mm to (187.8, 77.5), turned to -168 degrees
- moved D27 8.68 mm to (194.9, 110.7), turned to -168 degrees
- moved SW35 8.67 mm to (195.2, 133.8), turned to 12 degrees
- moved D35 8.61 mm to (200.8, 138.4), turned to -168 degrees
- moved SW26 8.44 mm to (172.2, 111.8), turned to 12 degrees
- moved D26 8.37 mm to (177.7, 116.4), turned to -168 degrees
- moved SW16 8.27 mm to (168.6, 95.2), turned to 12 degrees
- moved D17 8.24 mm to (191.3, 94.1), turned to -168 degrees
- moved D16 8.18 mm to (174.1, 99.8), turned to -168 degrees
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Connections:
- D1 pad 1: col0 -> row0
- D10 pad 1: col0 -> row0
- D11 pad 1: col1 -> row1
- D12 pad 1: col1 -> row1
- D13 pad 1: col1 -> row1
- D14 pad 1: col1 -> row1
- D15 pad 1: col1 -> row1
- D16 pad 1: col1 -> row1
- D17 pad 1: col1 -> row1
- D18 pad 1: col1 -> row1
- D19 pad 1: col1 -> row1
- D2 pad 1: col0 -> row0
- D20 pad 1: col1 -> row1
- D21 pad 1: col2 -> row2
- D22 pad 1: col2 -> row2
- D23 pad 1: col2 -> row2
- D24 pad 1: col2 -> row2
- D25 pad 1: col2 -> row2
- D26 pad 1: col2 -> row2
- D27 pad 1: col2 -> row2
- D28 pad 1: col2 -> row2
- D29 pad 1: col2 -> row2
- D3 pad 1: col0 -> row0
- D30 pad 1: col2 -> row2
- D31 pad 1: col3 -> row3
- D32 pad 1: col3 -> row3
- D33 pad 1: col3 -> row3
- D34 pad 1: col3 -> row3
- D35 pad 1: col3 -> row3
- D36 pad 1: col3 -> row3
- D4 pad 1: col0 -> row0
- D5 pad 1: col0 -> row0
- D6 pad 1: col0 -> row0
- D7 pad 1: col0 -> row0
- D8 pad 1: col0 -> row0
- D9 pad 1: col0 -> row0
- SW1 pad 2: row0 -> col0
- SW11 pad 2: row0 -> col0
- SW12 pad 2: row1 -> col1
- SW13 pad 2: row2 -> col2
- SW14 pad 2: row3 -> col3
- SW15 pad 2: row4 -> col4
- SW16 pad 2: row5 -> col5
- SW17 pad 2: row6 -> col6
- SW18 pad 2: row7 -> col7
- SW19 pad 2: row8 -> col8
- SW2 pad 2: row1 -> col1
- SW21 pad 2: row0 -> col0
- SW22 pad 2: row1 -> col1
- SW23 pad 2: row2 -> col2
- SW24 pad 2: row3 -> col3
- SW25 pad 2: row4 -> col4
- SW26 pad 2: row5 -> col5
- SW27 pad 2: row6 -> col6
- SW28 pad 2: row7 -> col7
- SW29 pad 2: row8 -> col8
- SW3 pad 2: row2 -> col2
- SW31 pad 2: row0 -> col0
- SW32 pad 2: row3 -> col3
- SW33 pad 2: row4 -> col4
- SW34 pad 2: row5 -> col5
- SW35 pad 2: row6 -> col6
- SW4 pad 2: row3 -> col3
- SW5 pad 2: row4 -> col4
- SW6 pad 2: row5 -> col5
- SW7 pad 2: row6 -> col6
- SW8 pad 2: row7 -> col7
- SW9 pad 2: row8 -> col8
- U1 pad 11: row2 -> row0
- U1 pad 15: row9 -> unconnected-(U1-Pad15)
- U1 pad 16: row8 -> unconnected-(U1-Pad16)
- U1 pad 17: row7 -> unconnected-(U1-Pad17)
- U1 pad 18: row6 -> unconnected-(U1-Pad18)
- U1 pad 19: row5 -> unconnected-(U1-Pad19)
- U1 pad 20: row4 -> unconnected-(U1-Pad20)
- U1 pad 5: col0 -> unconnected-(U1-Pad5)
- U1 pad 6: col1 -> unconnected-(U1-Pad6)
- U1 pad 7: col2 -> unconnected-(U1-Pad7)
- U1 pad 8: col3 -> unconnected-(U1-Pad8)
- U1 pad 9: row0 -> row2
Routing:
- net row3: track 0.00 -> 331.5 mm
- net row0: track 0.00 -> 331.4 mm
- net row1: track 0.00 -> 304.7 mm
- net row2: track 0.00 -> 277.1 mm
- net col0: track 0.00 -> 66.0 mm
- net col1: track 0.00 -> 65.6 mm, vias 0 -> 2
- net col4: track 0.00 -> 41.9 mm
- net row9: track 0.00 -> 41.9 mm
- net col6: track 0.00 -> 41.9 mm
- net col3: track 0.00 -> 41.9 mm
- net col5: track 0.00 -> 41.9 mm
- net col8: track 0.00 -> 31.4 mm
- net col7: track 0.00 -> 31.4 mm
- net col2: track 0.00 -> 31.4 mm
- net Net-(D21-Pad2): track 0.00 -> 14.6 mm
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Other:
- board outline added: 216.4 x 114 mm

Commit message: soweit so gut ENDGAME outline und layout final
Parts:
- moved SW_POWER1 4.49 mm to (133.3, 59.0)
- moved RSW1 4.49 mm to (143.1, 57.7)
- moved J2 4.49 mm to (158.2, 58.9)
- moved U1 3.92 mm to (145.3, 126.7)
- moved SW36 2.25 mm to (236.9, 132.0)
- moved SW16 2.25 mm to (166.4, 95.2)
- moved SW26 2.25 mm to (169.9, 111.9)
- moved SW6 2.25 mm to (162.8, 78.6)
- moved SW20 2.24 mm to (241.4, 85.5)
- moved SW10 2.24 mm to (241.4, 68.5)
- moved SW30 2.24 mm to (241.4, 102.5)
- moved SW9 2.24 mm to (219.2, 65.6)
- moved SW29 2.24 mm to (222.8, 99.4)
- moved SW19 2.24 mm to (221.0, 82.5)
- moved SW8 2.24 mm to (198.3, 65.2)
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Connections:
- SW10 pad 2: row9 -> col9
- SW20 pad 2: row9 -> col9
- SW30 pad 2: row9 -> col9
- SW36 pad 2: row9 -> col9
- U1 pad 13: unconnected-(U1-Pad13) -> col0
- U1 pad 14: unconnected-(U1-Pad14) -> col1
- U1 pad 15: unconnected-(U1-Pad15) -> col2
- U1 pad 16: unconnected-(U1-Pad16) -> col3
- U1 pad 17: unconnected-(U1-Pad17) -> col4
- U1 pad 18: unconnected-(U1-Pad18) -> col5
- U1 pad 19: unconnected-(U1-Pad19) -> col6
- U1 pad 20: unconnected-(U1-Pad20) -> col7
- U1 pad 7: unconnected-(U1-Pad7) -> col9
- U1 pad 8: unconnected-(U1-Pad8) -> col8
Routing:
- net row3: track 331.5 -> 0.00 mm
- net row0: track 331.4 -> 0.00 mm
- net row1: track 304.7 -> 0.00 mm
- net row2: track 277.1 -> 0.00 mm
- net row9: track 41.9 -> 0.00 mm
- net col9: track 0.00 -> 41.9 mm
- net col1: track 65.6 -> 31.4 mm, vias 2 -> 0
- net col3: track 41.9 -> 57.8 mm
- net col2: track 31.4 -> 47.3 mm
- net col6: track 41.9 -> 57.8 mm
- net col4: track 41.9 -> 57.8 mm
- net col8: track 31.4 -> 47.3 mm
- net col0: track 66.0 -> 57.8 mm
- net col7: track 31.4 -> 36.9 mm
- net Net-(D35-Pad2): track 11.7 -> 15.9 mm
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Other:
- board size 216.4 x 114 mm -> 216 x 117.2 mm

Commit message: backup cause things can happen
Parts:
- moved D14 0.40 mm to (112.7, 96.9)
- moved SW27 0.40 mm to (187.4, 106.4)
- moved D25 0.40 mm to (126.3, 119.2)
- moved D7 0.40 mm to (188.0, 77.5)
- moved D8 0.40 mm to (206.1, 70.1)
- moved SW9 0.40 mm to (219.6, 65.8)
- moved SW16 0.40 mm to (166.7, 95.5)
- moved SW4 0.40 mm to (111.0, 73.1)
- moved D18 0.40 mm to (209.0, 86.9)
- moved D22 0.40 mm to (74.1, 106.2)
- moved SW5 0.40 mm to (128.2, 78.8)
- moved D5 0.40 mm to (133.4, 86.0)
- moved SW10 0.40 mm to (241.8, 68.7)
- moved D12 0.40 mm to (75.9, 89.3)
- moved SW23 0.40 mm to (86.9, 98.9)
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Routing:
- net col0: track 57.8 -> 113.2 mm
- net col9: track 41.9 -> 87.5 mm
- net col5: track 41.9 -> 79.5 mm
- net col1: track 31.4 -> 69.0 mm
- net col7: track 36.9 -> 69.0 mm
- net col8: track 47.3 -> 77.0 mm
- net col4: track 57.8 -> 79.5 mm
- net col2: track 47.3 -> 69.0 mm
- net col6: track 57.8 -> 79.5 mm
- net col3: track 57.8 -> 79.5 mm
Other:
- board size 216 x 117.2 mm -> 216 x 118.2 mm

Commit message: updates updates upddfkjds
Parts:
- RSW1: footprint Button_Switch_THT:SW_PUSH_6mm -> Button_Switch_SMD:SW_SPST_TL3342; moved to B.Cu
- moved SW_POWER1 22.2 mm to (155.8, 58.0), turned to 0 degrees
- moved J2 13.0 mm to (145.6, 58.5)
- moved RSW1 8.20 mm to (135.3, 58.9), turned to 180 degrees
- moved D29 0.53 mm to (230.3, 105.4)
- moved SW19 0.53 mm to (221.3, 83.3)
- moved SW5 0.53 mm to (128.2, 79.4)
- moved D3 0.53 mm to (98.2, 72.9)
- moved D17 0.53 mm to (191.5, 94.7)
- moved SW34 0.53 mm to (171.3, 139.4)
- moved D14 0.53 mm to (112.7, 97.4)
- moved SW30 0.53 mm to (241.8, 103.3)
- moved SW32 0.53 mm to (98.0, 134.8)
- moved D34 0.53 mm to (179.0, 143.8)
- moved D13 0.53 mm to (95.3, 89.7)
- moved D6 0.53 mm to (170.8, 83.8)
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Connections:
- U1 pad 10: row1 -> col7
- U1 pad 11: row0 -> col8
- U1 pad 12: row3 -> col9
- U1 pad 18: col5 -> row2
- U1 pad 19: col6 -> row1
- U1 pad 20: col7 -> row0
- U1 pad 7: col9 -> row3
- U1 pad 8: col8 -> col5
- U1 pad 9: row2 -> col6
Routing:
- net row3: track 0.00 -> 216.3 mm
- net col5: track 79.5 -> 287.5 mm, vias 0 -> 1
- net col4: track 79.5 -> 277.8 mm, vias 0 -> 1
- net col6: track 79.5 -> 273.6 mm, vias 0 -> 1
- net col3: track 79.5 -> 259.0 mm, vias 0 -> 1
- net col7: track 69.0 -> 242.1 mm
- net col9: track 87.5 -> 249.1 mm
- net col2: track 69.0 -> 228.3 mm
- net col8: track 77.0 -> 232.7 mm
- net col1: track 69.0 -> 212.3 mm
- net col0: track 113.2 -> 206.4 mm
- net gnd: track 0.00 -> 77.7 mm
- net reset: track 0.00 -> 77.7 mm
- net raw: track 0.00 -> 72.7 mm
- net BT+: track 0.00 -> 11.7 mm
Other:
- outline, holes or cut-outs redrawn

Commit message: ja ja push den scheis
Parts:
- J2: footprint Connector_JST:JST_SH_BM02B-SRSS-TB_1x02-1MP_P1.00mm_Vertical -> Connector_JST:JST_PH_S2B-PH-K_1x02_P2.00mm_Horizontal
- RSW1: moved to F.Cu
- moved RSW1 89.3 mm to (132.0, 148.2)
- moved SW_POWER1 37.0 mm to (119.4, 51.3)
- moved J2 34.8 mm to (111.6, 51.0)
- moved D19 1.73 mm to (226.8, 88.8)
- moved D8 1.73 mm to (204.4, 71.0)
- moved D18 1.73 mm to (207.3, 87.8)
- moved D22 1.73 mm to (72.5, 107.1)
- moved D23 1.73 mm to (90.6, 106.8)
- moved D27 1.73 mm to (193.4, 111.7)
- moved SW28 1.73 mm to (202.8, 99.8)
- moved D10 1.73 mm to (246.6, 75.5)
- moved D2 1.73 mm to (76.0, 73.3)
- moved D25 1.73 mm to (124.6, 120.1)
- moved D5 1.73 mm to (131.7, 86.8)
- moved SW10 1.73 mm to (240.1, 69.6)
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Connections:
- U1 pad 18: row2 -> unconnected-(U1-Pad18)
- U1 pad 19: row1 -> unconnected-(U1-Pad19)
- U1 pad 2: unconnected-(U1-Pad2) -> row0
- U1 pad 20: row0 -> unconnected-(U1-Pad20)
- U1 pad 5: unconnected-(U1-Pad5) -> row1
- U1 pad 6: unconnected-(U1-Pad6) -> row2
Routing:
- net row1: track 0.00 -> 210.0 mm
- net row2: track 0.00 -> 199.3 mm
- net row0: track 0.00 -> 195.8 mm
- net gnd: track 77.7 -> 139.5 mm, vias 0 -> 1
- net reset: track 77.7 -> 38.5 mm, vias 0 -> 1
- net col0: track 206.4 -> 226.9 mm
- net raw: track 72.7 -> 86.0 mm, vias 0 -> 1
- net col8: track 232.7 -> 222.3 mm
- net col9: track 249.1 -> 240.0 mm
- net row3: track 216.3 -> 220.6 mm
- net col7: track 242.1 -> 239.8 mm
- net col6: track 273.6 -> 271.5 mm
- net col1: track 212.3 -> 211.1 mm
- net col2: track 228.3 -> 227.2 mm
- net col3: track 259.0 -> 258.0 mm
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Other:
- outline, holes or cut-outs redrawn

Commit message: back das up baby
Parts:
- moved D18 1.70 mm to (209.0, 87.9)
- moved D29 1.70 mm to (230.3, 105.9)
- moved SW1 1.70 mm to (49.6, 69.8)
- moved D13 1.70 mm to (95.3, 90.2)
- moved SW25 1.70 mm to (121.1, 113.1)
- moved D6 1.70 mm to (170.8, 84.3)
- moved D28 1.70 mm to (212.0, 104.7)
- moved D11 1.70 mm to (56.1, 92.7)
- moved SW9 1.70 mm to (219.6, 66.9)
- moved SW14 1.70 mm to (107.5, 90.8)
- moved SW28 1.70 mm to (204.5, 100.0)
- moved D17 1.70 mm to (191.5, 95.2)
- moved D26 1.70 mm to (177.9, 117.6)
- moved D34 1.70 mm to (179.0, 144.4)
- moved D20 1.70 mm to (248.3, 92.7)
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Connections:
- U1 pad 2: row0 -> row2
- U1 pad 6: row2 -> row0
Routing:
- net row2: track 199.3 -> 423.6 mm
- net row0: track 195.8 -> 397.7 mm
- net row1: track 210.0 -> 407.6 mm
- added copper zone on B.Cu, net gnd
- added copper zone on F.Cu, net gnd
Other:
- outline, holes or cut-outs redrawn

Commit message: biba backup
Parts:
- D1, D10, D11, D12, D13, D14, D15, D16, D17, D18, D19, D2, D20, D21, D22, D23, D24, D25, D26, D27, D28, D29, D3, D30, D31, D32, D33, D34, D35, D36, D4, D5, D6, D7, D8, D9: footprint Diode_SMD:D_SOD-123 -> Diode_SMD:D_SOD-123 CLEAN
- SW1, SW10, SW11, SW12, SW13, SW14, SW15, SW16, SW17, SW18, SW19, SW2, SW20, SW21, SW22, SW23, SW24, SW25, SW26, SW27, SW28, SW29, SW3, SW30, SW31, SW32, SW33, SW34, SW35, SW36, SW4, SW5, SW6, SW7, SW8, SW9: footprint keyswitches:Kailh_socket_PG1350_optional -> keyswitches:Kailh_socket_PG1350_optional_CLEAN
- moved D16 2.64 mm to (171.9, 101.8)
- moved D25 2.64 mm to (123.8, 121.2)
- moved D36 2.64 mm to (241.4, 140.1)
- moved D8 2.64 mm to (203.6, 72.1)
- moved SW10 2.64 mm to (239.3, 70.7)
- moved SW16 2.64 mm to (164.2, 97.4)
- moved SW35 2.64 mm to (190.9, 136.2)
- moved D23 2.64 mm to (89.8, 107.9)
- moved D26 2.64 mm to (175.4, 118.5)
- moved D30 2.64 mm to (245.9, 110.6)
- moved D9 2.64 mm to (224.2, 73.0)
- moved SW27 2.64 mm to (185.0, 108.4)
- moved U1 2.64 mm to (143.2, 128.9)
- moved SW14 2.64 mm to (105.0, 91.7)
- moved D14 2.64 mm to (110.2, 98.9)
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Routing:
- net row1: track 407.6 -> 391.2 mm
- net row2: track 423.6 -> 407.4 mm
- net row0: track 397.7 -> 382.2 mm
- net raw: track 86.0 -> 79.2 mm
- net row3: track 220.6 -> 216.1 mm
- net gnd: track 139.5 -> 139.6 mm, vias 1 -> 12
Other:
- board size 216 x 118.2 mm -> 216 x 114.2 mm
